File: connectors.kicad_sch (KiCad schematic)
At the start: 6 parts, among them J10 Conn_01x05_Pin, J11 Conn_01x05_Pin, J12 Conn_01x07_Pin, J13 Conn_02x04_Counter_Clockwise, J14 Conn_02x04_Counter_Clockwise, J9 Conn_01x05_Pin

Commit message: added load switches
Parts:
- J10, J11, J9: footprint (none) -> Connector_PinHeader_2.00mm:PinHeader_1x05_P2.00mm_Vertical
- J12: footprint (none) -> Connector_PinHeader_2.00mm:PinHeader_1x07_P2.00mm_Vertical
- J13, J14: footprint (none) -> Connector_PinHeader_2.00mm:PinHeader_2x04_P2.00mm_Vertical
Changed lines of the file:
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@@
 			)
 		)
-		(property "Footprint" ""
+		(property "Footprint" "Connector_PinHeader_2.00mm:PinHeader_1x07_P2.00mm_Vertical"
 			(at 36.83 55.88 0)
 			(effects
@@
 			)
 		)
-		(property "Footprint" ""
+		(property "Footprint" "Connector_PinHeader_2.00mm:PinHeader_2x04_P2.00mm_Vertical"
 			(at 78.74 55.88 0)
 			(effects
@@
 			)
 		)
-		(property "Footprint" ""
+		(property "Footprint" "Connector_PinHeader_2.00mm:PinHeader_1x05_P2.00mm_Vertical"
 			(at 34.29 25.4 0)
 			(effects
@@
 			)
 		)
-		(property "Footprint" ""
+		(property "Footprint" "Connector_PinHeader_2.00mm:PinHeader_2x04_P2.00mm_Vertical"
 			(at 114.3 54.61 0)
 			(effects
@@
 			)
 		)
-		(property "Footprint" ""
+		(property "Footprint" "Connector_PinHeader_2.00mm:PinHeader_1x05_P2.00mm_Vertical"
 			(at 76.2 25.4 0)
 			(effects
@@
 			)
 		)
-		(property "Footprint" ""
+		(property "Footprint" "Connector_PinHeader_2.00mm:PinHeader_1x05_P2.00mm_Vertical"
 			(at 119.38 25.4 0)
 			(effects

Commit message: save before sdram redesign
Parts:
- removed J10, J11, J9: Conn_01x05_Pin, Connector_PinHeader_2.00mm:PinHeader_1x05_P2.00mm_Vertical, symbol Connector:Conn_01x05_Pin
- removed J12: Conn_01x07_Pin, Connector_PinHeader_2.00mm:PinHeader_1x07_P2.00mm_Vertical, symbol Connector:Conn_01x07_Pin
- added J1, J2, J9: Conn_01x04_Pin, Connector_PinHeader_2.00mm:PinHeader_1x04_P2.00mm_Vertical, symbol Connector:Conn_01x04_Pin
- added J10: Conn_01x06_Pin, Connector_PinHeader_2.00mm:PinHeader_1x06_P2.00mm_Vertical, symbol Connector:Conn_01x06_Pin
Connections:
- net +3.3V: now also J1.4 (Pin_4), J10.6 (Pin_6), J2.4 (Pin_4), J9.4 (Pin_4)
- net GND: now also J1.1 (Pin_1), J10.1 (Pin_1), J2.1 (Pin_1), J9.1 (Pin_1)
- net LPI2C4_SCL: now also J1.3 (Pin_3)
- net LPI2C4_SDA: now also J1.2 (Pin_2)
- net LPSPI4_CS: now also J10.5 (Pin_5)
- net LPSPI4_SCK: now also J10.2 (Pin_2)
- net LPSPI4_SDI: now also J10.4 (Pin_4)
- net LPSPI4_SDO: now also J10.3 (Pin_3)
- net LPUART2_RX: now also J9.2 (Pin_2)
- net LPUART2_TX: now also J9.3 (Pin_3)
- net LPUART3_RX: now also J2.2 (Pin_2)
- net LPUART3_TX: now also J2.3 (Pin_3)
