File: hoperf.kicad_sch (KiCad schematic)
At the start: 3 parts, among them J8 Conn_Coaxial_Small, U5 RFM98W-433S2

Commit message: added load switches
Parts:
- R12: footprint Resistor_SMD:R_0603_1608Metric -> Resistor_SMD:R_0402_1005Metric
Changed lines of the file:
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@@
 			)
 		)
-		(property "Footprint" "Resistor_SMD:R_0603_1608Metric"
+		(property "Footprint" "Resistor_SMD:R_0402_1005Metric"
 			(at 39.37 35.56 0)
 			(effects

Commit message: save before sdram redesign
Parts:
- J8: footprint Connector_Coaxial:SMA_Amphenol_132289_EdgeMount -> Connector_Coaxial:SMA_Amphenol_132134_Vertical
- U5: footprint (none) -> footprints:HOPERF_RFM95W_SMD
Changed lines of the file:
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@@
+			)
+		)
+		(property "Flight" ""
+			(at 39.37 35.56 0)
+			(effects
+				(font
+					(size 1.27 1.27)
+				)
+				(hide yes)
+			)
+		)
+		(property "Proto" ""
+			(at 39.37 35.56 0)
+			(effects
+				(font
+					(size 1.27 1.27)
+				)
+				(hide yes)
 			)
 		)
@@
 			)
 		)
-		(property "Footprint" "Connector_Coaxial:SMA_Amphenol_132289_EdgeMount"
+		(property "Footprint" "Connector_Coaxial:SMA_Amphenol_132134_Vertical"
 			(at 104.14 35.56 0)
 			(effects
@@
 		)
 		(property "Description" "small coaxial connector (BNC, SMA, SMB, SMC, Cinch/RCA, LEMO, ...)"
+			(at 104.14 35.56 0)
+			(effects
+				(font
+					(size 1.27 1.27)
+				)
+				(hide yes)
+			)
+		)
+		(property "Flight" ""
+			(at 104.14 35.56 0)
+			(effects
+				(font
+					(size 1.27 1.27)
+				)
+				(hide yes)
+			)
+		)
+		(property "Proto" ""
 			(at 104.14 35.56 0)
 			(effects
@@
 			)
 		)
-		(property "Footprint" ""
+		(property "Footprint" "footprints:HOPERF_RFM95W_SMD"
 			(at -10.16 1.27 0)
 			(effects
@@
 			(at 73.66 43.18 0)
 			(effects
+				(font
+					(size 1.27 1.27)
+				)
+				(hide yes)
+			)
+		)
+		(property "Flight" ""
+			(at 73.66 43.18 0)
+			(effects
+				(font
+					(size 1.27 1.27)
+				)
+				(hide yes)
+			)
+		)
+		(property "Proto" ""
+			(at 73.66 43.18 0)
+			(effects
