File: spe.kicad_sch (KiCad schematic)
At the start: 6 parts, among them U2 DP83TC813SRHFRQ1

Commit message: finished v1
Parts:
- added C55, C56: 100n, symbol Device:C_Small
- added C57: 4.7n, symbol Device:C_Small
- added FL1: DLW32MH201XK2L, DLW32MH101XK2L, symbol DLW32MH201XK2L:DLW32MH201XK2L
- added J7: Conn_01x02, symbol Connector_Generic:Conn_01x02
- added R10, R9: 1k, symbol Device:R_Small_US
- added R11: 100k, symbol Device:R_Small_US
Connections:
- net GND: now also C57.1, R11.2
- net TRD_P: now reaches U2.19 (TRD_P)
- net TRD_P: now also FL1.3
- net TRD_M: now reaches U2.20 (TRD_M)
- net TRD_M: now also FL1.2
- new net: C55.1, FL1.1
- new net: C55.2, J7.1 (Pin_1), R9.1
- new net: C56.1, FL1.4
- new net: C56.2, J7.2 (Pin_2), R10.1
- new net: C57.2, R10.2, R11.1, R9.2
Other:
- company: (none) -> Northeastern University
- title: (none) -> RT1050 DevBoard for Project Horizon
- moved on the sheet: C45, C46, C47, C48, C49, U2

Commit message: added load switches
Parts:
- added U11: TPS22921YZPR, YZP6, symbol TPS22921:TPS22921YZPR
- C45, C46, C47, C48, C49, C55, C56, C57: footprint (none) -> Capacitor_SMD:C_0402_1005Metric
- J7: footprint (none) -> Connector_JST:JST_SH_BM02B-SRSS-TB_1x02-1MP_P1.00mm_Vertical
- R10, R11, R9: footprint (none) -> Resistor_SMD:R_0402_1005Metric
Connections:
- net +3.3V: now also U11.A2 (VIN), U11.B2 (VIN); no longer C45.1, C46.1, C47.1, C48.1, C49.1, U2.15 (VLSEEP), U2.18 (VDDA), U2.23 (VDDMAC), U2.7 (VDDIO)
- net GND: now also U11.C1 (GND)
- new net SPE_SWITCH: U11.C2 (ON)
- new net SPE_V: C45.1, C46.1, C47.1, C48.1, C49.1, U11.A1 (VOUT), U11.B1 (VOUT), U2.15 (VLSEEP), U2.18 (VDDA), U2.23 (VDDMAC), U2.7 (VDDIO)

Commit message: save before sdram redesign
Parts:
- C45, C46, C47, C48, C49, C55, C56, C57: footprint Capacitor_SMD:C_0402_1005Metric -> Capacitor_SMD:C_0201_0603Metric
- J7: footprint Connector_JST:JST_SH_BM02B-SRSS-TB_1x02-1MP_P1.00mm_Vertical -> Connector_JST:JST_PH_B2B-PH-K_1x02_P2.00mm_Vertical
