File: spe.kicad_sch (KiCad schematic)
At the start: 15 parts, among them J7 Conn_01x02, U11 TPS22921YZPR, U2 DP83TC813SRHFRQ1

Commit message: changes to board due to availability of components
Parts:
- C55, C56: value 100n -> 100nF
Changed lines of the file:
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@@
 			)
 		)
-		(property "Value" "100n"
+		(property "Value" "100nF"
 			(at 95.2563 95.25 90)
 			(effects
@@
 			)
 		)
-		(property "Value" "100n"
+		(property "Value" "100nF"
 			(at 95.2563 106.68 90)
 			(effects
