File: usb_debug.kicad_sch (KiCad schematic)
At the start: 19 parts, among them J5 USB_C_Receptacle_USB2.0, SW1 SW_DIP_x02, U1 MIMXRT1052CVJ5B, U7 PRTR5V0U2X, U8 XC6206P332PR-G

Commit message: quick fix
Parts:
- C32: footprint Capacitor_SMD:C_0201_0603Metric -> Capacitor_SMD:C_0402_1005Metric
Changed lines of the file:
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@@
 			)
 		)
-		(property "Footprint" "Capacitor_SMD:C_0201_0603Metric"
+		(property "Footprint" "Capacitor_SMD:C_0402_1005Metric"
 			(at 43.18 53.34 0)
 			(effects
