File: mcu_power.kicad_sch (KiCad schematic)
At the start: 36 parts, among them U1 MIMXRT1052CVJ5B, Y1 DSC1001BI5-024.0000, Y2 830107834801

Commit message: quick fix
Parts:
- C28: footprint Capacitor_SMD:C_0201_0603Metric -> Capacitor_SMD:C_0603_1608Metric
Changed lines of the file:
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@@
 			)
 		)
-		(property "Footprint" "Capacitor_SMD:C_0201_0603Metric"
+		(property "Footprint" "Capacitor_SMD:C_0603_1608Metric"
 			(at 182.88 146.05 0)
 			(effects

Commit message: changes to board due to availability of components
Parts:
- L1: footprint Inductor_SMD:L_0402_1005Metric -> Inductor_SMD:L_0603_1608Metric
Changed lines of the file:
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@@
 			)
 		)
-		(property "Footprint" "Inductor_SMD:L_0402_1005Metric"
+		(property "Footprint" "Inductor_SMD:L_0603_1608Metric"
 			(at 173.99 129.54 0)
 			(effects
